Commit message: Reading robot URDF from param robot_state_publisher/robot_description. Fixed errors at on_configure.

File: description/urdf/ur5_description.urdf.xacro (robot description, xacro)
@@ -218,7 +218,10 @@
     </collision>
     <inertial>
-      <mass value="0"/>
-      <origin rpy="0 0 0" xyz="0 0 0"/>
-      <inertia ixx="0" ixy="0" ixz="0" iyy="0" iyz="0" izz="0"/>
+      <mass value="0.134"/>
+      <origin rpy="0 0 0" xyz="-0.01 0.0 0.0"/>
+      <inertia
+        ixx="0.012" ixy="0" ixz="0"
+        iyy="0.012" iyz="0"
+        izz="0.024"/>
     </inertial>
   </link>

Commit message: Fix inertia values. New values from ros-industrial/universal_robot

File: description/urdf/ur5_description.urdf.xacro (robot description, xacro)
@@ -23,5 +23,5 @@
     </collision>
     <inertial>
-      <mass value="4.0"/>
+      <mass value="4.0000"/>
       <origin rpy="0 0 0" xyz="0.0 0.0 0.0"/>
       <inertia
@@ -52,10 +52,10 @@
     </collision>
     <inertial>
-      <mass value="3.7"/>
-      <origin rpy="0 0 0" xyz="0.0 0.0 0.0"/>
-      <inertia
-        ixx="0.010267495893" ixy="0.0" ixz="0.0"
-        iyy="0.010267495893" iyz="0.0"
-        izz="0.00666"/>
+      <mass value="3.7000"/>
+      <origin rpy="0 0 0" xyz="0.0 0.0 0.0"/>
+      <inertia
+        ixx="0.014972358333333331" ixy="0.0" ixz="0.0"
+        iyy="0.014972358333333331" iyz="0.0"
+        izz="0.01040625"/>
     </inertial>
   </link>
@@ -81,9 +81,9 @@
     </collision>
     <inertial>
-      <mass value="8.393"/>
+      <mass value="8.3930"/>
       <origin rpy="0 0 0" xyz="0.0 0.0 0.28"/>
       <inertia
-        ixx="0.22689067591" ixy="0.0" ixz="0.0"
-        iyy="0.22689067591" iyz="0.0"
+        ixx="0.13388583541666665" ixy="0.0" ixz="0.0"
+        iyy="0.13388583541666665" iyz="0.0"
         izz="0.0151074"/>
     </inertial>
@@ -110,9 +110,9 @@
     </collision>
     <inertial>
-      <mass value="2.275"/>
+      <mass value="2.3300"/>
       <origin rpy="0 0 0" xyz="0.0 0.0 0.25"/>
       <inertia
-        ixx="0.049443313556" ixy="0.0" ixz="0.0"
-        iyy="0.049443313556" iyz="0.0"
+        ixx="0.031216803515624995" ixy="0.0" ixz="0.0"
+        iyy="0.031216803515624995" iyz="0.0"
         izz="0.004095"/>
     </inertial>
@@ -139,10 +139,10 @@
     </collision>
     <inertial>
-      <mass value="1.219"/>
-      <origin rpy="0 0 0" xyz="0.0 0.0 0.0"/>
-      <inertia
-        ixx="0.111172755531" ixy="0.0" ixz="0.0"
-        iyy="0.111172755531" iyz="0.0"
-        izz="0.21942"/>
+      <mass value="1.2190"/>
+      <origin rpy="0 0 0" xyz="0.0 0.0 0.0"/>
+      <inertia
+        ixx="0.002013889583333333" ixy="0.0" ixz="0.0"
+        iyy="0.002013889583333333" iyz="0.0"
+        izz="0.0021942"/>
     </inertial>
   </link>
@@ -168,10 +168,10 @@
     </collision>
     <inertial>
-      <mass value="1.219"/>
-      <origin rpy="0 0 0" xyz="0.0 0.0 0.0"/>
-      <inertia
-        ixx="0.111172755531" ixy="0.0" ixz="0.0"
-        iyy="0.111172755531" iyz="0.0"
-        izz="0.21942"/>
+      <mass value="1.2190"/>
+      <origin rpy="0 0 0" xyz="0.0 0.0 0.0"/>
+      <inertia
+        ixx="0.0018310395833333333" ixy="0.0" ixz="0.0"
+        iyy="0.0018310395833333333" iyz="0.0"
+        izz="0.0021942"/>
     </inertial>
   </link>
@@ -197,10 +197,10 @@
     </collision>
     <inertial>
-      <mass value="0.1879"/>
-      <origin rpy="0 0 0" xyz="0.0 0.0 0.0"/>
-      <inertia
-        ixx="0.0171364731454" ixy="0.0" ixz="0.0"
-        iyy="0.0171364731454" iyz="0.0"
-        izz="0.033822"/>
+      <mass value="0.18790"/>
+      <origin rpy="0 0 0" xyz="0.0 0.0 0.0"/>
+      <inertia
+        ixx="8.062475833333332e-05" ixy="0.0" ixz="0.0"
+        iyy="8.062475833333332e-05" iyz="0.0"
+        izz="0.0001321171875"/>
     </inertial>
   </link>
@@ -210,20 +210,5 @@
     <origin rpy="0.0 0.0 1.57079632679" xyz="0.0 0.0823 0.0"/>
   </joint>
-  <link name="ee_link">
-    <collision>
-      <geometry>
-        <box size="0.01 0.01 0.01"/>
-      </geometry>
-      <origin rpy="0 0 0" xyz="-0.01 0 0"/>
-    </collision>
-    <inertial>
-      <mass value="0.134"/>
-      <origin rpy="0 0 0" xyz="-0.01 0.0 0.0"/>
-      <inertia
-        ixx="0.012" ixy="0" ixz="0"
-        iyy="0.012" iyz="0"
-        izz="0.024"/>
-    </inertial>
-  </link>
+  <link name="ee_link"/>
   </xacro:macro>
 </robot>
