Commit message: Add FT sensor to the robot description. Sensor not working on Gazebo

File: description/urdf/ur5.description.urdf.xacro (robot description, xacro)
@@ -209,6 +209,38 @@
     <child link="ee_link"/>
     <origin rpy="0.0 0.0 1.57079632679" xyz="0.0 0.0823 0.0"/>
-  </joint>
-  <link name="ee_link"/>
+    <sensor name="force_torque_sensor" type="force_torque">
+      <update_rate>100</update_rate>
+      <always_on>true</always_on>
+      <visualize>true</visualize>
+      <topic>end_effector_ft</topic>
+      <force_torque>
+        <frame>sensor</frame>
+        <measure_direction>parent_to_child</measure_direction>
+      </force_torque>
+    </sensor>
+  </joint>
+  <link name="ee_link">
+  <!-- Bota Systems AG Rokubi FT sensor -->
+    <visual>
+      <geometry>
+        <cylinder radius="0.024" length="0.032" />
+      </geometry>
+      <origin rpy="0 1.57079632679 0" xyz="0.016 0.0 0.0"/>
+    </visual>
+    <collision>
+      <geometry>
+        <cylinder radius="0.024" length="0.032" />
+      </geometry>
+      <origin rpy="0 1.57079632679 0" xyz="0.016 0.0 0.0"/>
+    </collision>
+    <inertial>
+      <mass value="0.118"/>
+      <origin rpy="0 1.57079632679 0" xyz="0.016 0.0 0.0"/>
+      <inertia
+        ixx="8.00e-05" ixy="0.0" ixz="0.0"
+        iyy="8.00e-05" iyz="0.0"
+        izz="1.40e-04"/>
+    </inertial>
+  </link>
   </xacro:macro>
 </robot>

Commit message: Organize for v1.0.0

File: description/urdf/ur5.description.urdf.xacro (robot description, xacro)
@@ -243,5 +243,6 @@
     </collision>
     <inertial>
-      <mass value="0.118"/>
+      <!-- mass value="0.118"/ -->
+      <mass value="0.001"/>
       <origin rpy="0 1.57079632679 0" xyz="0.016 0.0 0.0"/>
       <inertia

Commit message: Diagnostic FT sensor noisy reading

File: description/urdf/ur5.description.urdf.xacro (robot description, xacro)
@@ -217,4 +217,7 @@
       </geometry>
       <origin rpy="0 1.57079632679 0" xyz="0.016 0.0 0.0"/>
+      <material name="Orange">
+        <color rgba="0.8 0.4 0.0 1.0"/>
+      </material>
     </visual>
     <collision name="sensor_body">

Commit message: Add FT sensor filtering and simplified collision geometries

File: description/urdf/ur5.description.urdf.xacro (robot description, xacro)
@@ -193,6 +193,7 @@
     <collision>
       <geometry>
-        <mesh filename="package://ros2_impedance_controller/description/meshes/ur5/collision/wrist3.stl"/>
-      </geometry>
+        <cylinder radius="0.037" length="0.035" />
+      </geometry>
+      <origin rpy="1.57079632679 0 0" xyz="0.0 0.065 0.0"/>
     </collision>
     <inertial>
@@ -214,5 +215,5 @@
     <visual>
       <geometry>
-        <cylinder radius="0.024" length="0.032" />
+        <cylinder radius="0.024" length="0.030" />
       </geometry>
       <origin rpy="0 1.57079632679 0" xyz="0.016 0.0 0.0"/>
@@ -223,29 +224,12 @@
     <collision name="sensor_body">
       <geometry>
-        <cylinder radius="0.024" length="0.026" />
-      </geometry>
-      <origin rpy="0 1.57079632679 0" xyz="0.019 0.0 0.0"/>
-    </collision>
-    <collision name="sensor_body_c1">
-      <geometry>
-        <sphere radius="0.006" />
-      </geometry>
-      <origin rpy="0 0 0" xyz="0.006 -0.02035159 -0.01175"/>
-    </collision>
-    <collision name="sensor_body_c2">
-      <geometry>
-        <sphere radius="0.006" />
-      </geometry>
-      <origin rpy="0 0 0" xyz="0.006 0.02035159 -0.01175"/>
-    </collision>
-    <collision name="sensor_body_c3">
-      <geometry>
-        <sphere radius="0.006" />
-      </geometry>
-      <origin rpy="0 0 0" xyz="0.006 0 0.0235"/>
+        <cylinder radius="0.024" length="0.030" />
+      </geometry>
+      <origin rpy="0 1.57079632679 0" xyz="0.016 0.0 0.0"/>
+      <max_contacts>6</max_contacts>
     </collision>
     <inertial>
       <!-- mass value="0.118"/ -->
-      <mass value="0.001"/>
+      <mass value="0.054"/>
       <origin rpy="0 1.57079632679 0" xyz="0.016 0.0 0.0"/>
       <inertia

Commit message: Add command filtering. Tuning is unstable for 'm_d = 0'

File: description/urdf/ur5.description.urdf.xacro (robot description, xacro)
@@ -37,5 +37,5 @@
     <axis xyz="0 0 1"/>
     <limit effort="150.0" lower="-6.28318530718" upper="6.28318530718" velocity="3.15"/>
-    <dynamics damping="0.33" friction="0.0"/>
+    <dynamics damping="0.20" friction="0.0"/>
   </joint>
   <link name="shoulder_link">
@@ -66,5 +66,5 @@
     <axis xyz="0 1 0"/>
     <limit effort="150.0" lower="-6.28318530718" upper="6.28318530718" velocity="3.15"/>
-    <dynamics damping="0.3" friction="0.0"/>
+    <dynamics damping="0.10" friction="0.0"/>
   </joint>
   <link name="upper_arm_link">
@@ -95,5 +95,5 @@
     <axis xyz="0 1 0"/>
     <limit effort="150.0" lower="-3.14159265359" upper="3.14159265359" velocity="3.15"/>
-    <dynamics damping="0.3" friction="0.0"/>
+    <dynamics damping="0.10" friction="0.0"/>
   </joint>
   <link name="forearm_link">
@@ -124,5 +124,5 @@
     <axis xyz="0 1 0"/>
     <limit effort="28.0" lower="-6.28318530718" upper="6.28318530718" velocity="3.2"/>
-    <dynamics damping="0.10" friction="0.0"/>
+    <dynamics damping="0.20" friction="0.0"/>
   </joint>
   <link name="wrist_1_link">
@@ -153,5 +153,5 @@
     <axis xyz="0 0 1"/>
     <limit effort="28.0" lower="-6.28318530718" upper="6.28318530718" velocity="3.2"/>
-    <dynamics damping="0.10" friction="0.0"/>
+    <dynamics damping="0.20" friction="0.0"/>
   </joint>
   <link name="wrist_2_link">
@@ -182,5 +182,5 @@
     <axis xyz="0 1 0"/>
     <limit effort="28.0" lower="-6.28318530718" upper="6.28318530718" velocity="3.2"/>
-    <dynamics damping="0.07" friction="0.0"/>
+    <dynamics damping="0.20" friction="0.0"/>
   </joint>
   <link name="wrist_3_link">
@@ -231,5 +231,5 @@
     <inertial>
       <!-- mass value="0.118"/ -->
-      <mass value="0.054"/>
+      <mass value="0.018"/>
       <origin rpy="0 1.57079632679 0" xyz="0.016 0.0 0.0"/>
       <inertia
