Commit message: Update wall position and size

File: description/environment/environment.xacro (robot description, xacro)
@@ -5,11 +5,12 @@
     <color rgba="${153/255} ${255/255} ${51/255} 0.67"/>
   </material>
-  <xacro:property name="mass" value="20.0" />
-  <xacro:property name="width" value="0.30" />
-  <xacro:property name="height" value="1.2" />
+  <xacro:property name="mass" value="10.0" />
+  <xacro:property name="width" value="0.160" />
+  <xacro:property name="length" value="1.20" />
+  <xacro:property name="height" value="1.00" />
   <joint name="wall_joint" type="fixed">
     <parent link="${world_link}"/>
     <child link="wall_link" />
-    <origin rpy="0.0 0.0 0.0" xyz="0.80 0.0 0.0"/>
+    <origin rpy="0.0 0.0 0.0" xyz="${0.55 + width/2} ${0.05 + length/2} 0.0"/>
   </joint>
   <link name="wall_link">
@@ -17,5 +18,5 @@
       <origin xyz="0 0 ${height/2}" rpy="0 0 0"/>
       <geometry>
-        <box size="${width} ${width} ${height}"/>
+        <box size="${width} ${length} ${height}"/>
       </geometry>
     </collision>
@@ -23,5 +24,5 @@
       <origin xyz="0 0 ${height/2}" rpy="0 0 0"/>
       <geometry>
-        <box size="${width} ${width} ${height}"/>
+        <box size="${width} ${length} ${height}"/>
       </geometry>
       <material name="greenyellow"/>
@@ -31,7 +32,7 @@
       <mass value="${mass}"/>
       <inertia
-        ixx="${mass / 12.0 * (width*width + height*height)}" ixy="0.0" ixz="0.0"
+        ixx="${mass / 12.0 * (length*length + height*height)}" ixy="0.0" ixz="0.0"
         iyy="${mass / 12.0 * (height*height + width*width)}" iyz="0.0"
-        izz="${mass / 12.0 * (width*width + width*width)}"/>
+        izz="${mass / 12.0 * (length*length + width*width)}"/>
     </inertial>
   </link>

Commit message: Debugging collision with the wall. Added Gazebo world file.

File: description/environment/environment.xacro (robot description, xacro)
@@ -1,5 +1,5 @@
 <?xml version="1.0"?>
 <robot xmlns:xacro="http://ros.org/wiki/xacro">
-  <xacro:macro name="environment" params="world_link">
+  <xacro:macro name="environment" params="parent_link">
   <material name="greenyellow">
     <color rgba="${153/255} ${255/255} ${51/255} 0.67"/>
@@ -10,5 +10,5 @@
   <xacro:property name="height" value="1.00" />
   <joint name="wall_joint" type="fixed">
-    <parent link="${world_link}"/>
+    <parent link="${parent_link}"/>
     <child link="wall_link" />
     <origin rpy="0.0 0.0 0.0" xyz="${0.55 + width/2} ${0.05 + length/2} 0.0"/>
@@ -20,4 +20,11 @@
         <box size="${width} ${length} ${height}"/>
       </geometry>
+      <surface>
+        <friction>
+          <ode/>
+        </friction>
+        <bounce/>
+        <contact/>
+      </surface>
     </collision>
     <visual>

File: description/urdf/ur5.urdf.xacro (robot description, xacro)
@@ -6,4 +6,11 @@
   <xacro:include filename="$(find ros2_impedance_controller)/description/environment/environment.xacro" />
   <link name="world"/>
+  <!-- Collision is not working with this URDF.
+       However, the collision settings are properly
+       defined on Gazebo, and it with for the ground
+       and added objects in Gazebo. Consider create
+       a world model then.
+  -->
+  <xacro:environment parent_link="world"/>
   <xacro:ur5_robot parent="world">
     <origin xyz="0 0 0" rpy="0 0 0" />
@@ -14,4 +21,3 @@
     <xacro:ur5_gazebo/>
   </xacro:if>
-  <xacro:environment world_link="world"/>
 </robot>
