Commit message: End-effector FT sensor working! Sensor output on gz topic.

File: description/gazebo/ur5.gazebo.xacro (robot description, xacro)
@@ -7,4 +7,17 @@
       </plugin>
     </gazebo>
+    <gazebo reference="ee_fixed_joint">
+      <provideFeedback>true</provideFeedback>
+      <preserveFixedJoint>true</preserveFixedJoint>
+      <sensor name="force_torque_sensor" type="force_torque">
+        <update_rate>100</update_rate>
+        <always_on>true</always_on>
+        <topic>end_effector_ft_sensor</topic>
+        <force_torque>
+          <frame>sensor</frame>
+          <measure_direction>child_to_parent</measure_direction>
+        </force_torque>
+      </sensor>
+    </gazebo>
   </xacro:macro>
 </robot>

File: description/urdf/ur5.description.urdf.xacro (robot description, xacro)
@@ -209,14 +209,4 @@
     <child link="ee_link"/>
     <origin rpy="0.0 0.0 1.57079632679" xyz="0.0 0.0823 0.0"/>
-    <sensor name="force_torque_sensor" type="force_torque">
-      <update_rate>100</update_rate>
-      <always_on>true</always_on>
-      <visualize>true</visualize>
-      <topic>end_effector_ft</topic>
-      <force_torque>
-        <frame>sensor</frame>
-        <measure_direction>parent_to_child</measure_direction>
-      </force_torque>
-    </sensor>
   </joint>
   <link name="ee_link">
@@ -228,9 +218,27 @@
       <origin rpy="0 1.57079632679 0" xyz="0.016 0.0 0.0"/>
     </visual>
-    <collision>
-      <geometry>
-        <cylinder radius="0.024" length="0.032" />
-      </geometry>
-      <origin rpy="0 1.57079632679 0" xyz="0.016 0.0 0.0"/>
+    <collision name="sensor_body">
+      <geometry>
+        <cylinder radius="0.024" length="0.026" />
+      </geometry>
+      <origin rpy="0 1.57079632679 0" xyz="0.019 0.0 0.0"/>
+    </collision>
+    <collision name="sensor_body_c1">
+      <geometry>
+        <sphere radius="0.006" />
+      </geometry>
+      <origin rpy="0 0 0" xyz="0.006 -0.02035159 -0.01175"/>
+    </collision>
+    <collision name="sensor_body_c2">
+      <geometry>
+        <sphere radius="0.006" />
+      </geometry>
+      <origin rpy="0 0 0" xyz="0.006 0.02035159 -0.01175"/>
+    </collision>
+    <collision name="sensor_body_c3">
+      <geometry>
+        <sphere radius="0.006" />
+      </geometry>
+      <origin rpy="0 0 0" xyz="0.006 0 0.0235"/>
     </collision>
     <inertial>
