Commit message: Enhance the states reading with ordered interfaces. Command interfaces are not working.

File: description/ros2_control/ur5.ros2_control.xacro (robot description, xacro)
@@ -1,6 +1,6 @@
 <?xml version="1.0"?>
 <robot xmlns:xacro="http://www.ros.org/wiki/xacro">
-  <xacro:macro name="ur5_control" params="name use_gazebo:=^|true">
-    <ros2_control name="${name}" type="system">
+  <xacro:macro name="ur5_control" params="use_gazebo:=^|true">
+    <ros2_control name="GazeboSimSystem" type="system">
       <hardware>
         <xacro:if value="${use_gazebo}">

File: description/urdf/ur5.urdf.xacro (robot description, xacro)
@@ -4,10 +4,9 @@
   <xacro:include filename="$(find ros2_impedance_controller)/description/urdf/ur5_description.urdf.xacro" />
   <xacro:include filename="$(find ros2_impedance_controller)/description/ros2_control/ur5.ros2_control.xacro" />
-  <!-- Used for fixing robot -->
   <link name="world"/>
   <xacro:ur5_robot parent="world">
     <origin xyz="0 0 0" rpy="0 0 0" />
   </xacro:ur5_robot>
-  <xacro:ur5_control name="UR5RobotSystem" use_gazebo="$(arg use_gazebo)"/>
+  <xacro:ur5_control use_gazebo="$(arg use_gazebo)"/>
   <xacro:if value="$(arg use_gazebo)">
     <xacro:include filename="$(find ros2_impedance_controller)/description/gazebo/ur5.gazebo.xacro" />

File: description/urdf/ur5_description.urdf.xacro (robot description, xacro)
@@ -37,5 +37,5 @@
     <axis xyz="0 0 1"/>
     <limit effort="150.0" lower="-6.28318530718" upper="6.28318530718" velocity="3.15"/>
-    <dynamics damping="0.0" friction="0.0"/>
+    <dynamics damping="0.33" friction="0.0"/>
   </joint>
   <link name="shoulder_link">
@@ -66,5 +66,5 @@
     <axis xyz="0 1 0"/>
     <limit effort="150.0" lower="-6.28318530718" upper="6.28318530718" velocity="3.15"/>
-    <dynamics damping="0.0" friction="0.0"/>
+    <dynamics damping="0.3" friction="0.0"/>
   </joint>
   <link name="upper_arm_link">
@@ -95,5 +95,5 @@
     <axis xyz="0 1 0"/>
     <limit effort="150.0" lower="-3.14159265359" upper="3.14159265359" velocity="3.15"/>
-    <dynamics damping="0.0" friction="0.0"/>
+    <dynamics damping="0.3" friction="0.0"/>
   </joint>
   <link name="forearm_link">
@@ -124,5 +124,5 @@
     <axis xyz="0 1 0"/>
     <limit effort="28.0" lower="-6.28318530718" upper="6.28318530718" velocity="3.2"/>
-    <dynamics damping="0.0" friction="0.0"/>
+    <dynamics damping="0.10" friction="0.0"/>
   </joint>
   <link name="wrist_1_link">
@@ -153,5 +153,5 @@
     <axis xyz="0 0 1"/>
     <limit effort="28.0" lower="-6.28318530718" upper="6.28318530718" velocity="3.2"/>
-    <dynamics damping="0.0" friction="0.0"/>
+    <dynamics damping="0.10" friction="0.0"/>
   </joint>
   <link name="wrist_2_link">
@@ -182,5 +182,5 @@
     <axis xyz="0 1 0"/>
     <limit effort="28.0" lower="-6.28318530718" upper="6.28318530718" velocity="3.2"/>
-    <dynamics damping="0.0" friction="0.0"/>
+    <dynamics damping="0.07" friction="0.0"/>
   </joint>
   <link name="wrist_3_link">

Commit message: Add robot yaml with joints initial postions

File: description/ros2_control/ur5.ros2_control.xacro (robot description, xacro)
@@ -2,4 +2,6 @@
 <robot xmlns:xacro="http://www.ros.org/wiki/xacro">
   <xacro:macro name="ur5_control" params="use_gazebo:=^|true">
+    <xacro:property name="robot_yaml" value="$(find ros2_impedance_controller)/config/robot.yaml"/>
+    <xacro:property name="config" value="${xacro.load_yaml(robot_yaml)}"/>
     <ros2_control name="UR5RobotSystem" type="system">
       <hardware>
@@ -15,5 +17,5 @@
         <command_interface name="effort"/>
         <state_interface name="position">
-          <param name="initial_value">1.189</param>
+          <param name="initial_value">${config['initial']['shoulder_pan']}</param>
         </state_interface>
         <state_interface name="velocity"/>
@@ -23,5 +25,5 @@
         <command_interface name="effort"/>
         <state_interface name="position">
-          <param name="initial_value">-1.800</param>
+          <param name="initial_value">${config['initial']['shoulder_lift']}</param>
         </state_interface>
         <state_interface name="velocity"/>
@@ -31,5 +33,5 @@
         <command_interface name="effort"/>
         <state_interface name="position">
-          <param name="initial_value">1.409</param>
+          <param name="initial_value">${config['initial']['elbow']}</param>
         </state_interface>
         <state_interface name="velocity"/>
@@ -39,5 +41,5 @@
         <command_interface name="effort"/>
         <state_interface name="position">
-          <param name="initial_value">0.373</param>
+          <param name="initial_value">${config['initial']['wrist_1']}</param>
         </state_interface>
         <state_interface name="velocity"/>
@@ -47,5 +49,5 @@
         <command_interface name="effort"/>
         <state_interface name="position">
-          <param name="initial_value">1.189</param>
+          <param name="initial_value">${config['initial']['wrist_2']}</param>
         </state_interface>
         <state_interface name="velocity"/>
@@ -55,5 +57,5 @@
         <command_interface name="effort"/>
         <state_interface name="position">
-          <param name="initial_value">0.0</param>
+          <param name="initial_value">${config['initial']['wrist_3']}</param>
         </state_interface>
         <state_interface name="velocity"/>
